File: BriefcaseAmp.kicad_pcb (KiCad board)
At the start: 2 copper layers, 10 parts, among them J2 XLR3_Switched, J5 AudioJack3_Switch, J6 AudioJack3_Switch, U1 TP4056, U2 TP4056, U3 TP4056, U4 TP4056, U5 TP4056, U6 TP4056, U7 LD1086V33-DG

Commit message: changes
Parts:
- removed J2: XLR3_Switched, Connector_Audio:Jack_XLR_Neutrik_NC5FAV_Vertical
- added BT1: Battery_Cell, Battery:BatteryHolder_MPD_BH-18650-PC2, B.Cu at (-22.9, 9.58)
- added BT2: Battery_Cell, Battery:BatteryHolder_MPD_BH-18650-PC2, B.Cu at (-25.5, 29.1)
- added BT3: Battery_Cell, Battery:BatteryHolder_MPD_BH-18650-PC2, B.Cu at (-25.5, 47.4)
- added BT4: Battery_Cell, Battery:BatteryHolder_MPD_BH-18650-PC2, B.Cu at (-27.5, 67.5)
- added BT5: Battery_Cell, Battery:BatteryHolder_MPD_BH-18650-PC2, B.Cu at (-27.2, 86.0)
- added BT6: Battery_Cell, Battery:BatteryHolder_MPD_BH-18650-PC2, B.Cu at (-27.2, 106.9)
- added C1: C_Polarized, Capacitor_THT:CP_Radial_D6.3mm_P2.50mm, F.Cu at (101.6, 95.0)
- added C2: C_Polarized, Capacitor_THT:CP_Radial_D6.3mm_P2.50mm, F.Cu at (113.5, 92.5)
- added J9: Power Inlet, Connector_PinHeader_2.54mm:PinHeader_1x04_P2.54mm_Horizontal, B.Cu at (91.7, 89.7)
- added PS1: IRM-05-5, Converter_ACDC:Converter_ACDC_MeanWell_IRM-05-xx_THT, F.Cu at (160.0, 138.9)
- added SW2: Enable Amp, Button_Switch_THT:SW_CuK_JS202011CQN_DPDT_Straight, F.Cu at (77.2, 96.5)
- J5: value AudioJack3_Switch -> Left
- J6: value AudioJack3_Switch -> Right
- moved U4 222.3 mm to (-85.5, 60.2)
- moved U5 222.3 mm to (-85.5, 78.6)
- moved U6 222.3 mm to (-85.5, 97.1)
- moved U1 222.3 mm to (-85.3, 1.02)
- moved U2 222.3 mm to (-85.4, 19.7)
- moved U3 222.3 mm to (-85.4, 38.4)
- moved J6 106.8 mm to (91.4, 148.1), turned to 180 degrees
- moved J5 63.5 mm to (91.3, 126.3), turned to 180 degrees
- moved U7 57.3 mm to (108.5, 89.9), turned to -90 degrees
Connections:
- net +12V renamed +12VA
- net -12V renamed -12VA
- U3 pad 4: GND -> GNDA
- U4 pad 3: GND -> GNDA
- U7 pad 1: unconnected-(U7-Pad1) -> GND
- U7 pad 2: unconnected-(U7-Pad2) -> +3V3
- U7 pad 3: unconnected-(U7-Pad3) -> Net-(C1-Pad1)
Routing:
- added copper zone on B.Cu, net GND
Other:
- board outline added: 119.1 x 65.3 mm
