File: BriefcaseAmp.kicad_sch (KiCad schematic)
At the start: 29 parts, among them J1 AC Inlet, J2 Conn_Coaxial_x2, J3 Conn_01x02, J4 Conn_01x02, J5 AudioJack3_Switch, J6 AudioJack3_Switch, SW1 SW_SPST, T1 Transformer_1P_SS, U1 TP4056, U2 TP4056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

Commit message: changes
Parts:
- added C1, C2: C_Polarized, Capacitor_THT:CP_Radial_D6.3mm_P2.50mm, symbol Device:C_Polarized
- added F1: Fuse, symbol Device:Fuse
- added J7: Conn_01x03, symbol Connector_Generic:Conn_01x03
- added J8: Power Outlet, symbol Connector_Generic:Conn_01x04
- added J9: Power Inlet, Connector_PinHeader_2.54mm:PinHeader_1x04_P2.54mm_Horizontal, symbol Connector_Generic:Conn_01x04
- added PS1: IRM-05-5, Converter_ACDC:Converter_ACDC_MeanWell_IRM-05-xx_THT, symbol Converter_ACDC:IRM-05-5
- added SW2: Enable Amp, Button_Switch_THT:SW_CuK_JS202011CQN_DPDT_Straight, symbol Switch:SW_Push_DPDT
- added SW3: AC / Battery, symbol Switch:SW_SPDT
- BT1, BT2, BT3, BT4, BT5, BT6: footprint (none) -> Battery:BatteryHolder_MPD_BH-18650-PC2
- J5: value AudioJack3_Switch -> Left
- J6: value AudioJack3_Switch -> Right
Connections:
- net +12V: now also J9.4 (Pin_4), SW2.2 (B); no longer U1.3 (OUT+)
- net -12V: now also J9.1 (Pin_1), SW2.5 (B); no longer U6.4 (OUT-)
- net AC: now also F1.2, PS1.2 (AC/L); no longer J1.2 (Pin_2)
- net GND: now also U7.1 (ADJ/GND), C1.2, C2.2, J7.2 (Pin_2), J9.2 (Pin_2), PS1.3 (-Vo); no longer U3.4 (OUT-), U4.3 (OUT+)
- net GNDPWR: now also PS1.1 (AC/N)
- net at U2.4 (OUT-), U3.3 (OUT+): now also J8.3 (Pin_3)
- net +3V3: now reaches U7.2 (OUT)
- net +3V3: now also C2.1
- net at U7.3 (IN): now also C1.1, SW3.2 (B)
- new net: F1.1, J1.2 (Pin_2)
- new net: J7.1 (Pin_1), SW2.1 (A)
- new net: J7.3 (Pin_3), SW2.6 (C)
- new net +12VA: J8.4 (Pin_4), U1.3 (OUT+)
- new net +4V: J9.3 (Pin_3), SW3.3 (C)
- new net +5V: PS1.4 (+Vo), SW3.1 (A)
- new net -12VA: J8.1 (Pin_1), U6.4 (OUT-)
- new net GNDA: J8.2 (Pin_2), U3.4 (OUT-), U4.3 (OUT+)
- no-connect marks 12 -> 20
Other:
- note added: "Red: +12V White: 4.2V Black: GND Yellow: -12V"
- note added: "what happens when the -17V feed back when the amp is AC powered?"
- moved on the sheet: BT1, D1, J1, J2, J3, J4, J5, J6, LS1, LS2, LS3, LS4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
